File: Hardware/MicroMod_Environmental.brd (EAGLE design)
At the start: 65 x 38 mm, 56 parts, among them J1 MICROMOD_STANDARD, U1 SGP40, U2 EEPROM, U3 SHTC3, U4 3.3V, U5 STC31

Commit message: Updates function board symbol to new one in the official SFE eagle library repo
Parts:
- J1: value MICROMOD_STANDARD -> MICROMOD_FUNCTION_STANDARD; device SparkFun-MicroMod-Function:M.2-CARD-E-22_FUNCTION_STANDARD -> SparkFun-MicroMod:M.2-CARD-E-22_FUNCTION_STANDARD
- R1, R2: value 2.2k -> 4.7k
Changed lines of the file:
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@@
 <?xml version="1.0" encoding="utf-8"?>
 <!DOCTYPE eagle SYSTEM "eagle.dtd">
-<eagle version="9.6.2">
+<eagle version="9.5.1">
 <drawing>
 <settings>
@@
 <attribute name="REV" value="" x="12.7" y="-17.78" size="1.778" layer="27" display="off"/>
 </element>
-<element name="J1" library="SparkFun-MicroMod-Function" package="M.2-CARD-E-22_FUNCTION_STANDARD" value="MICROMOD_STANDARD" x="0" y="19.05" smashed="yes" rot="R270"/>
-<element name="R1" library="SparkFun-Resistors" package="0603" value="2.2k" x="11.049" y="13.081" smashed="yes" rot="R270">
+<element name="J1" library="SparkFun-MicroMod" package="M.2-CARD-E-22_FUNCTION_STANDARD" value="MICROMOD_FUNCTION_STANDARD" x="0" y="19.05" smashed="yes" rot="R270"/>
+<element name="R1" library="SparkFun-Resistors" package="0603" value="4.7k" x="11.049" y="13.081" smashed="yes" rot="R270">
 <attribute name="NAME" x="11.811" y="13.081" size="0.6096" layer="25" font="vector" ratio="20" rot="R270" align="bottom-center"/>
-<attribute name="PROD_ID" value="RES-08272" x="11.049" y="13.081" size="1.778" layer="27" font="vector" ratio="15" rot="R270" display="off"/>
-<attribute name="VALUE" value="2.2k" x="10.287" y="13.081" size="0.6096" layer="27" font="vector" ratio="20" rot="R270" align="top-center"/>
+<attribute name="PROD_ID" value="RES-07857" x="11.049" y="13.081" size="1.778" layer="27" font="vector" ratio="15" rot="R270" display="off"/>
+<attribute name="VALUE" x="10.287" y="13.081" size="0.6096" layer="27" font="vector" ratio="20" rot="R270" align="top-center"/>
 </element>
-<element name="R2" library="SparkFun-Resistors" package="0603" value="2.2k" x="9.017" y="13.081" smashed="yes" rot="R270">
+<element name="R2" library="SparkFun-Resistors" package="0603" value="4.7k" x="9.017" y="13.081" smashed="yes" rot="R270">
 <attribute name="NAME" x="9.779" y="13.081" size="0.6096" layer="25" font="vector" ratio="20" rot="R270" align="bottom-center"/>
-<attribute name="PROD_ID" value="RES-08272" x="9.017" y="13.081" size="1.778" layer="27" font="vector" ratio="15" rot="R270" display="off"/>
-<attribute name="VALUE" value="2.2k" x="8.255" y="13.081" size="0.6096" layer="27" font="vector" ratio="20" rot="R270" align="top-center"/>
+<attribute name="PROD_ID" value="RES-07857" x="9.017" y="13.081" size="1.778" layer="27" font="vector" ratio="15" rot="R270" display="off"/>
+<attribute name="VALUE" x="8.255" y="13.081" size="0.6096" layer="27" font="vector" ratio="20" rot="R270" align="top-center"/>
 </element>
 <element name="C5" library="SparkFun-Capacitors" package="0603" value="1.0uF" x="16.637" y="31.242" smashed="yes" rot="R90">
